File: RP2040-LBX.kicad_pcb (KiCad board)
At the start: 2 copper layers, 292.7 x 140.6 mm, 65 parts, among them J1 USB C Connector, J2 JTAG_TC2030, U1 XC6206, U2 USBLC6-2SC6, U3 RP2040, U4 W25Q128JVS, Y1 12MHz

Commit message: fix: some routing; moved tactiles a bit
Parts:
- moved SW_BOOTSEL1 0.71 mm to (131.4, 62.4)
- moved SW_HOME1 0.71 mm to (121.9, 62.4)
- moved SW_L3 0.71 mm to (112.5, 62.4)
- moved SW_PSTOUCH1 0.71 mm to (103.1, 62.4)
- moved SW_R3 0.71 mm to (93.6, 62.4)
Routing:
- net SW_L3: track 112.0 -> 118.7 mm
- net SW_PSTOUCH: track 127.6 -> 128.3 mm
- net USB_BOOT: track 80.4 -> 81.1 mm
- net SW_HOME: track 108.4 -> 109.1 mm
- net SW_R3: track 137.2 -> 137.9 mm

Commit message: fix: edge cuts smaller to fit any case
Parts:
- moved R1 1.00 mm to (206.9, 65.5)
- moved R2 1.00 mm to (198.4, 66.3)
- moved R3 1.00 mm to (202.3, 66.3)
- moved J1 1.00 mm to (200.4, 58.5)
Routing:
- net 3vCable: track 107.5 -> 106.8 mm
- net DBUS-: track 45.4 -> 46.0 mm
Other:
- board size 292.7 x 140.6 mm -> 290.7 x 139.1 mm
